File: Tank/Tank/untitled.sch (EAGLE design)
At the start: 37 parts, among them U1 L298N, U2 Atmega1284, U3 Regulator 6V, U4 Regulator 5v, X1 Led RGB, X10 Encoder Dreapta, X12 Switch power, X13 Switch reset, X14 Senzor distanta 2, X15 Senzor distanta 3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

Commit message: laptop->pc test part
Parts:
- removed C3: 100nF, Passives:CAPACITORTHT_2.54
- R5, R9: device Passives:RESISTORTHT_5.08 -> Passives:RESISTORTHT_2.54
- U1: value L298N -> L298NMULTIWATT15V_PERFBOARD; device Motors:L298N -> Motors:L298NMULTIWATT15V_PERFBOARD
- X11: value (none) -> Middle battery
- X8: value (none) -> High battery
- X9: value (none) -> Low battery
Connections:
- net EN_A_PWM renamed EN_D_PWM
- net EN_B_PWM renamed EN_S_PWM
- removed net B_RX: R5.P$1, R5.P$2, R6.P$2, U2.PD1, X4.4
- removed net N$37: X11.1, X8.2
- new net B_ON: R3.P$2, U2.PB2
- new net B_RX_3V3: R5.P$1, R6.P$2, X4.4
- new net B_RX_5V: R5.P$2, U2.PD1
- new net G_ON: R2.P$2, U2.PB1
- new net LED_PWM: R4.P$2, U2.PD5
- new net N$2: X11.2, X8.1
- new net R_ON: R1.P$2, U2.PB0
- new net VBATT: X12.2, X8.2
- net B: no longer R3.P$2, U2.PB2
- net D1: now also U2.PC4; no longer U2.PA5
- net D2: now also U2.PC2; no longer U2.PA6
- net D3: now also U2.PA5; no longer U2.PA7
- net EN_REG: now also U2.PA2; no longer U2.PD3
- net G: no longer R2.P$2, U2.PB1
- net GND: now also X10.4, X6.4, X7.5, X9.1; no longer C3.P$2, X10.1, X6.1, X7.6, X9.2
- net IN_1: now also U2.PC7; no longer U2.PC0
- net IN_2: now also U2.PC6; no longer U2.PC1
- net IN_3: now also U2.PC5; no longer U2.PC2
- net L_PWM: no longer R4.P$2, U2.PD5
- net M1_D: now also U1.OUT_1; no longer U1.OUT_2
- net M1_S: now also X6.3; no longer X6.6
- net M2_D: now also U1.OUT_2; no longer U1.OUT_1
- net M2_S: now also X6.2; no longer X6.5
- net N$43: now also X11.1, X9.2; no longer X11.2, X9.1
- net OUTA_D: now also U2.PA7; no longer U2.PC4
- net OUTA_S: now also U2.PC1, X6.6; no longer U2.PC6, X6.3
- net OUTB_D: now also U2.PA6; no longer U2.PC5
- net OUTB_S: now also U2.PC0, X6.5; no longer U2.PC7, X6.2
- net R: no longer R1.P$2, U2.PB0
- net RESET: now also X7.6; no longer X7.4
- net VCC5V: now also X10.1, X6.1, X7.4; no longer C3.P$1, X10.4, X6.4, X7.5
- net VIN11V: no longer X12.2, X8.1
Other:
- moved on the sheet: R1, R2, R3, R4, X1, X11, X2, X8, X9
